File: picov.kicad_pcb (KiCad board)
At the start: 2 copper layers, 21.2 x 51.3 mm, 35 parts, among them J1 USB_C_Receptacle_USB2.0_16P, J2 Conn_01x20, J3 Conn_01x20, J4 Conn_01x03, SW1 Boot, SW2 Reset, SW3 SW_Push, U1 RP2040, U2 AP2112K-3.3, U3 W25Q16JVUXIQ_TR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

Commit message: Finished all design for the pcb
Parts:
- SW1, SW2, SW3: footprint Button_Switch_SMD:SW_Push_SPST_NO_Alps_SKRK -> Button_Switch_SMD:SW_SPST_CK_KXT3
- moved C10 67.2 mm to (191.1, 55.1)
- moved C9 64.8 mm to (190.8, 56.5), turned to 90 degrees
- moved C14 55.8 mm to (183.7, 58.7)
- moved SW3 47.9 mm to (187.6, 89.3)
- moved C16 47.4 mm to (185.4, 81.0), turned to 90 degrees
- moved C15 40.9 mm to (182.4, 83.4), turned to 180 degrees
- moved R7 36.1 mm to (184.5, 88.0)
- moved SW2 35.2 mm to (185.3, 85.4), turned to 90 degrees
- moved D1 14.8 mm to (189.3, 53.4), turned to 180 degrees
- moved R3 12.0 mm to (187.4, 51.3), turned to 90 degrees
- moved R6 9.94 mm to (181.8, 58.7), turned to 180 degrees
- moved U3 3.89 mm to (182.0, 61.8), turned to 90 degrees
- moved C13 2.72 mm to (186.3, 80.6)
- moved C6 2.27 mm to (181.8, 67.6), turned to -90 degrees
- moved U2 1.73 mm to (188.7, 56.6)
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Connections:
- net Net-(U1-USB_DM) renamed FN
- net Net-(U1-USB_DP) renamed FP
- U4 pad 1: USBDP -> USBDN
- U4 pad 3: USBDN -> USBDP
- U4 pad 4: CLEAN_USBDN -> CLEAN_USBDP
- U4 pad 5: +5V -> VSYS
- U4 pad 6: CLEAN_USBDP -> CLEAN_USBDN
Routing:
- net +3V3: track 41.2 -> 84.1 mm, vias 7 -> 8
- net IO0: track 0.00 -> 27.7 mm
- net IO1: track 0.00 -> 25.7 mm
- net RUN: track 0.00 -> 24.6 mm, vias 0 -> 3
- net VSYS: track 0.00 -> 22.9 mm
- net IO15: track 0.00 -> 21.3 mm
- net IO2: track 0.00 -> 21.2 mm
- net IO23: track 0.00 -> 20.9 mm, vias 0 -> 2
- net +5V: track 0.00 -> 20.6 mm
- net IO16: track 0.00 -> 20.5 mm
- net IO3: track 0.00 -> 19.4 mm
- net SWCLK: track 0.00 -> 19.1 mm
- net IO14: track 0.00 -> 18.6 mm
- net SWD: track 0.00 -> 18.1 mm
- net IO17: track 0.00 -> 18.1 mm
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- added copper zone on B.Cu, net GND
- added copper zone on F.Cu, net GND
- removed copper zone on B.Cu, net (none)
- removed copper zone on F.Cu, net (none)
Other:
- board text added: "3V3"
- board text added: "BOOT"
- board text added: "GND"
- board text added: "IO0"
- board text added: "IO1"
- board text added: "IO10"
- board text added: "IO11"
- board text added: "IO12"
- board text added: "IO13"
- board text added: "IO14"
- board text added: "IO15"
- board text added: "IO16"
- board text added: "IO17"
- board text added: "IO18"
- board text added: "IO19"
- board text added: "IO2"
- board text added: "IO20"
- board text added: "IO21"
- board text added: "IO22"
- board text added: "IO23"
- board text added: "IO26"
- board text added: "IO27"
- board text added: "IO28"
- board text added: "IO3"
- board text added: "IO4"
- board text added: "IO5"
- board text added: "IO6"
- board text added: "IO7"
- board text added: "IO8"
- board text added: "IO9"
- board text added: "NC"
- board text added: "RST"
- board text added: "RUN"
- board text added: "VBUS"
- board text added: "VSYS"
