File: src/picov.kicad_sch (KiCad schematic)
At the start: 35 parts, among them J1 USB_C_Receptacle_USB2.0_16P, J2 Conn_01x20, J3 Conn_01x20, J4 Conn_01x03, SW1 Boot, SW2 Reset, SW3 SW_Push, U1 RP2040, U2 AP2112K-3.3, U3 W25Q16JVUXIQ_TR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

Commit message: finished pcb!
Parts:
- removed C9: 1uF, Capacitor_SMD:C_0402_1005Metric, symbol Device:C
- removed U2: AP2112K-3.3, Package_TO_SOT_SMD:SOT-23-5, symbol Regulator_Linear:AP2112K-3.3
- added C7: 10uF, Capacitor_SMD:C_0402_1005Metric, symbol Device:C
- added J5: Conn_01x06, Package_TO_SOT_SMD:SOT-23-6, symbol Connector_Generic:Conn_01x06
- added U10, U11, U5, U6, U7, U8, U9: WS2812-2020, WS2812-2020:LED_WS2812-2020, symbol WS2812-2020:WS2812-2020
- C10: value 1uF -> 10uF
- SW1: value Boot -> SW_Push; footprint Button_Switch_SMD:SW_Tactile_SPST_NO_Straight_CK_PTS636Sx25SMTRLFS -> Button_Switch_SMD:SMD_3x4; LCSC C2858607 -> C455280
- SW2: value Reset -> SW_Push; footprint Button_Switch_SMD:SW_SPST_CK_KXT3 -> Button_Switch_SMD:SMD_3x4; LCSC C2858607 -> C455280
- SW3: footprint Button_Switch_SMD:SW_SPST_CK_KXT3 -> Button_Switch_SMD:SMD_3x4; LCSC C2858607 -> C455280
- U3: footprint W25Q16JVUXIQ_TR:IC_W25Q16JVUXIQ_TR -> Package_SON:Winbond_USON-8-1EP_3x2mm_P0.5mm_EP0.2x1.6mm
Connections:
- net +3V3: now also J5.1 (Pin_1)
- net GND: now also J5.2 (Pin_2), U10.2 (GND), U11.2 (GND), U5.2 (GND), U6.2 (GND), U7.2 (GND), U8.2 (GND), U9.2 (GND)
- net IO25: now also U5.3 (DI)
- net VSYS: now also J5.3 (Pin_3), J5.5 (Pin_5), U10.4 (VDD), U11.4 (VDD), U5.4 (VDD), U6.4 (VDD), U7.4 (VDD), U8.4 (VDD), U9.4 (VDD)
- new net: U8.1 (DO), U9.3 (DI)
- new net: U7.1 (DO), U8.3 (DI)
- new net: C7.1, J5.4 (Pin_4)
- new net: C7.2, J5.6 (Pin_6)
- new net: U10.3 (DI), U9.1 (DO)
- new net: U10.1 (DO), U11.3 (DI)
- new net: U5.1 (DO), U6.3 (DI)
- new net: U6.1 (DO), U7.3 (DI)
- no-connect marks 4 -> 5
