File: src/picov.kicad_sch (KiCad schematic)
At the start: 42 parts, among them J1 USB_C_Receptacle_USB2.0_16P, J2 Conn_01x20, J3 Conn_01x20, J4 Conn_01x03, J5 Conn_01x06, SW1 SW_Push, SW2 SW_Push, SW3 SW_Push, U1 RP2040, U10 WS2812-2020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

Commit message: removed castellated holes due to high jlcpcb pricing, finished 4x4 neopixel matrix
Parts:
- removed SW3: SW_Push, Button_Switch_SMD:SMD_3x4, symbol Switch:SW_Push
- added U12, U13, U14, U15, U16, U17, U18, U19, U2: WS2812-2020, WS2812-2020:LED_WS2812-2020, symbol WS2812-2020:WS2812-2020
- C10, C7: LCSC C52923 -> C15525
- J2, J3: footprint Connector_PinHeader_2.54mm:Castellated_20 -> Connector_PinHeader_2.54mm:PinHeader_1x20_P2.54mm_Vertical; now in the parts list
- J4: now in the parts list
- U10, U11, U5, U6, U7, U8, U9: LCSC C965555 -> C26159668
Connections:
- net GND: now also U12.2 (GND), U13.2 (GND), U14.2 (GND), U15.2 (GND), U16.2 (GND), U17.2 (GND), U18.2 (GND), U19.2 (GND), U2.2 (GND)
- net IO23: now also U13.3 (DI)
- net IO24: now also U2.3 (DI)
- net IO29: now also U12.3 (DI)
- net VSYS: now also U12.4 (VDD), U13.4 (VDD), U14.4 (VDD), U15.4 (VDD), U16.4 (VDD), U17.4 (VDD), U18.4 (VDD), U19.4 (VDD), U2.4 (VDD)
- net at U8.1 (DO): no longer U9.3 (DI)
- new net: U17.1 (DO), U19.3 (DI)
- new net: U15.1 (DO), U17.3 (DI)
- new net: U13.1 (DO), U15.3 (DI)
- new net: U14.1 (DO), U16.3 (DI)
- new net: U12.1 (DO), U14.3 (DI)
- new net: U16.1 (DO), U18.3 (DI)
- new net: U2.1 (DO), U9.3 (DI)
- no-connect marks 5 -> 8

Commit message: changed some routing
Connections:
- net CLEAN_USBDN is gone; now on net USBDN: R2.2, U4.6 (I/O1)
- net CLEAN_USBDP is gone; now on net USBDP: R1.1, U4.4 (I/O2)
Changed lines of the file:
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@@
 		)
 	)
-	(global_label "CLEAN_USBDP"
+	(global_label "USBDP"
 		(shape input)
 		(at 134.62 41.91 0)
@@
 		)
 		(property "Intersheetrefs" "${INTERSHEET_REFS}"
-			(at 150.789 41.91 0)
+			(at 143.9552 41.91 0)
 			(effects
 				(font
@@
 		)
 	)
-	(global_label "CLEAN_USBDP"
+	(global_label "USBDP"
 		(shape input)
 		(at 201.93 58.42 90)
@@
 		)
 		(property "Intersheetrefs" "${INTERSHEET_REFS}"
-			(at 201.93 42.251 90)
+			(at 201.93 49.0848 90)
 			(effects
 				(font
@@
 		)
 	)
-	(global_label "CLEAN_USBDN"
+	(global_label "USBDN"
 		(shape input)
 		(at 134.62 39.37 0)
@@
 		)
 		(property "Intersheetrefs" "${INTERSHEET_REFS}"
-			(at 150.8495 39.37 0)
+			(at 144.0157 39.37 0)
 			(effects
 				(font
@@
 		)
 	)
-	(global_label "CLEAN_USBDN"
+	(global_label "USBDN"
 		(shape input)
 		(at 201.93 60.96 270)
@@
 		)
 		(property "Intersheetrefs" "${INTERSHEET_REFS}"
-			(at 201.93 77.1895 90)
-			(effects
-				(font
+			(at 201.93 70.3557 90)
+			(effects
+				(font
